File: scheme/KiCAD-shcemes/sum-diff-device/sum-diff-device.kicad_sch (KiCad schematic)
At the start: 52 parts, among them J1 Conn_01x08_Female, J2 Conn_01x08_Female, J3 SUM_DIFF, J4 Conn_01x08_Male, J5 Conn_01x02_Male, U1 SN74HC86N, U10 SN74HC08N, U11 SN74HC08N, U12 SN74HC27N, U13 SN74HC27N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

Commit message: feat: Created build for jlcpcb.
Parts:
- U1, U2, U3, U4, U5, U6: footprint footprints:DIP794W45P254L1969H508Q14 -> DIP794W45P254L1969H508Q14; symbol SN74HC86N:SN74HC86N -> Digital:SN74HC86N
- U10, U11, U16, U17, U7, U8, U9: footprint footprints:DIP794W45P254L1969H508Q14 -> DIP794W45P254L1969H508Q14; symbol SN74HC08N:SN74HC08N -> Digital:SN74HC08N
- U12, U13: footprint footprints:DIP794W45P254L1969H508Q14 -> DIP794W45P254L1969H508Q14; symbol SN74HC27N:SN74HC27N -> Digital:SN74HC27N
- U14: footprint footprints:DIP794W45P254L1969H508Q14 -> DIP794W45P254L1969H508Q14; symbol SN74HC05N:SN74HC05N -> Digital:SN74HC05N
- U15: footprint footprints:DIP794W45P254L1969H508Q14 -> DIP794W45P254L1969H508Q14; symbol SN74HC32N:SN74HC32N -> Digital:SN74HC32N

Commit message: feat: Added Enum with commands.
Parts:
- U1, U2, U3, U4, U5, U6: symbol Digital:SN74HC86N -> digital:SN74HC86N
- U10, U11, U16, U17, U7, U8, U9: symbol Digital:SN74HC08N -> digital:SN74HC08N
- U12, U13: symbol Digital:SN74HC27N -> digital:SN74HC27N
- U14: symbol Digital:SN74HC05N -> digital:SN74HC05N
- U15: symbol Digital:SN74HC32N -> digital:SN74HC32N
Changed lines of the file:
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@@
     (pin "1")
   )
-  (symbol (lib_id "Digital:SN74HC27N") (at 392.43 179.07 0) (unit 1)
+  (symbol (lib_id "digital:SN74HC27N") (at 392.43 179.07 0) (unit 1)
     (in_bom yes) (on_board yes) (fields_autoplaced)
     (property "Reference" "U12" (id 0) (at 392.43 153.67 0))
@@
     (pin "1")
   )
-  (symbol (lib_id "Digital:SN74HC32N") (at 643.89 107.95 0) (unit 1)
+  (symbol (lib_id "digital:SN74HC32N") (at 643.89 107.95 0) (unit 1)
     (in_bom yes) (on_board yes) (fields_autoplaced)
     (property "Reference" "U15" (id 0) (at 643.89 85.09 0))
@@
     (pin "1")
   )
-  (symbol (lib_id "Digital:SN74HC08N") (at 290.83 427.99 0) (unit 1)
+  (symbol (lib_id "digital:SN74HC08N") (at 290.83 427.99 0) (unit 1)
     (in_bom yes) (on_board yes) (fields_autoplaced)
     (property "Reference" "U11" (id 0) (at 290.83 405.13 0))
@@
     (pin "2")
   )
-  (symbol (lib_id "Digital:SN74HC86N") (at 120.65 238.76 0) (unit 1)
+  (symbol (lib_id "digital:SN74HC86N") (at 120.65 238.76 0) (unit 1)
     (in_bom yes) (on_board yes) (fields_autoplaced)
     (property "Reference" "U2" (id 0) (at 120.65 215.9 0))
@@
     (pin "8")
   )
-  (symbol (lib_id "Digital:SN74HC08N") (at 711.2 144.78 0) (unit 1)
+  (symbol (lib_id "digital:SN74HC08N") (at 711.2 144.78 0) (unit 1)
     (in_bom yes) (on_board yes) (fields_autoplaced)
     (property "Reference" "U16" (id 0) (at 711.2 121.92 0))
@@
     (pin "8")
   )
-  (symbol (lib_id "Digital:SN74HC08N") (at 290.83 302.26 0) (unit 1)
+  (symbol (lib_id "digital:SN74HC08N") (at 290.83 302.26 0) (unit 1)
     (in_bom yes) (on_board yes) (fields_autoplaced)
     (property "Reference" "U9" (id 0) (at 290.83 279.4 0))
@@
     (pin "2")
   )
-  (symbol (lib_id "Digital:SN74HC27N") (at 392.43 240.03 0) (unit 1)
+  (symbol (lib_id "digital:SN74HC27N") (at 392.43 240.03 0) (unit 1)
     (in_bom yes) (on_board yes) (fields_autoplaced)
     (property "Reference" "U13" (id 0) (at 392.43 214.63 0))
@@
     (pin "9")
   )
-  (symbol (lib_id "Digital:SN74HC86N") (at 200.66 173.99 0) (unit 1)
+  (symbol (lib_id "digital:SN74HC86N") (at 200.66 173.99 0) (unit 1)
     (in_bom yes) (on_board yes) (fields_autoplaced)
     (property "Reference" "U5" (id 0) (at 200.66 151.13 0))
@@
     (pin "1")
   )
-  (symbol (lib_id "Digital:SN74HC05N") (at 511.81 173.99 0) (unit 1)
+  (symbol (lib_id "digital:SN74HC05N") (at 511.81 173.99 0) (unit 1)
     (in_bom yes) (on_board yes) (fields_autoplaced)
     (property "Reference" "U14" (id 0) (at 511.81 153.67 0))
@@
     (pin "2")
   )
-  (symbol (lib_id "Digital:SN74HC86N") (at 120.65 175.26 0) (unit 1)
+  (symbol (lib_id "digital:SN74HC86N") (at 120.65 175.26 0) (unit 1)
     (in_bom yes) (on_board yes) (fields_autoplaced)
     (property "Reference" "U1" (id 0) (at 120.65 152.4 0))
@@
     (pin "2")
   )
-  (symbol (lib_id "Digital:SN74HC08N") (at 290.83 237.49 0) (unit 1)
+  (symbol (lib_id "digital:SN74HC08N") (at 290.83 237.49 0) (unit 1)
     (in_bom yes) (on_board yes) (fields_autoplaced)
     (property "Reference" "U8" (id 0) (at 290.83 214.63 0))
@@
     (pin "1")
   )
-  (symbol (lib_id "Digital:SN74HC08N") (at 290.83 364.49 0) (unit 1)
+  (symbol (lib_id "digital:SN74HC08N") (at 290.83 364.49 0) (unit 1)
     (in_bom yes) (on_board yes) (fields_autoplaced)
     (property "Reference" "U10" (id 0) (at 290.83 341.63 0))
@@
     (pin "1")
   )
-  (symbol (lib_id "Digital:SN74HC08N") (at 290.83 173.99 0) (unit 1)
+  (symbol (lib_id "digital:SN74HC08N") (at 290.83 173.99 0) (unit 1)
     (in_bom yes) (on_board yes) (fields_autoplaced)
     (property "Reference" "U7" (id 0) (at 290.83 151.13 0))
@@
     (pin "2")
   )
-  (symbol (lib_id "Digital:SN74HC86N") (at 120.65 368.3 0) (unit 1)
+  (symbol (lib_id "digital:SN74HC86N") (at 120.65 368.3 0) (unit 1)
     (in_bom yes) (on_board yes) (fields_autoplaced)
     (property "Reference" "U4" (id 0) (at 120.65 345.44 0))
@@
     (pin "1")
   )
-  (symbol (lib_id "Digital:SN74HC86N") (at 120.65 304.8 0) (unit 1)
+  (symbol (lib_id "digital:SN74HC86N") (at 120.65 304.8 0) (unit 1)
     (in_bom yes) (on_board yes) (fields_autoplaced)
     (property "Reference" "U3" (id 0) (at 120.65 281.94 0))
@@
     (pin "1")
   )
-  (symbol (lib_id "Digital:SN74HC08N") (at 711.2 198.12 0) (unit 1)
+  (symbol (lib_id "digital:SN74HC08N") (at 711.2 198.12 0) (unit 1)
     (in_bom yes) (on_board yes) (fields_autoplaced)
     (property "Reference" "U17" (id 0) (at 711.2 175.26 0))
@@
     (pin "1")
   )
-  (symbol (lib_id "Digital:SN74HC86N") (at 200.66 238.76 0) (unit 1)
+  (symbol (lib_id "digital:SN74HC86N") (at 200.66 238.76 0) (unit 1)
     (in_bom yes) (on_board yes)
     (property "Reference" "U6" (id 0) (at 200.66 215.9 0))
