File: scheme/KiCAD-shcemes/sum-diff-device/_autosave-sum-diff-device.kicad_sch (KiCad schematic)
At the start: 52 parts, among them J1 Conn_01x08_Female, J2 Conn_01x08_Female, J3 SUM_DIFF, J4 Conn_01x08_Male, J5 Conn_01x02_Male, U1 SN74HC86N, U10 SN74HC08N, U11 SN74HC08N, U12 SN74HC27N, U13 SN74HC27N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

Commit message: feat: Changed pcb for sum-diff device
Parts:
- J5: footprint (none) -> Connector_PinSocket_2.54mm:PinSocket_1x02_P2.54mm_Vertical
Changed lines of the file:
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@@
       (effects (font (size 1.27 1.27)) (justify left))
     )
-    (property "Footprint" "" (id 2) (at 167.64 21.59 0)
+    (property "Footprint" "Connector_PinSocket_2.54mm:PinSocket_1x02_P2.54mm_Vertical" (id 2) (at 167.64 21.59 0)
       (effects (font (size 1.27 1.27)) hide)
     )
@@
     )
     (path "/b30847d0-f930-472b-8921-bf45f226495b"
-      (reference "J5") (unit 1) (value "Conn_01x02_Male") (footprint "")
+      (reference "J5") (unit 1) (value "Conn_01x02_Male") (footprint "Connector_PinSocket_2.54mm:PinSocket_1x02_P2.54mm_Vertical")
     )
     (path "/b2848e41-fcd7-404b-a35a-7adb29400d55"
